Commit message: Diff Drive & URDF Added

File: ros_ws/src/sumo/urdf/gazebo.xacro (robot description, xacro)
@@ -10,5 +10,5 @@
       <pose relative_to="lidar_link">0 0 0 0 0 0</pose>
       <topic>scan</topic>
-      <update_rate>2</update_rate>
+      <update_rate>1</update_rate>
       <visualize>true</visualize>
       <lidar>
@@ -34,3 +34,61 @@
     </sensor>
   </gazebo>
+  <gazebo reference="camera_link">
+  <sensor name="camera_sensor" type="camera">
+    <always_on>true</always_on>
+    <visualize>true</visualize>
+    <update_rate>30</update_rate>
+    <camera>
+      <horizontal_fov>1.5708</horizontal_fov>
+      <image>
+        <width>1280</width>
+        <height>720</height>
+        <format>R8G8B8</format>
+      </image>
+      <clip>
+        <near>0.05</near>
+        <far>100.0</far>
+      </clip>
+    </camera>
+    <topic>camera/image</topic>
+  </sensor>
+</gazebo>
+<gazebo>
+  <plugin
+      filename="gz-sim-diff-drive-system"
+      name="gz::sim::systems::DiffDrive">
+    <left_joint>front_left_wheel_joint</left_joint>
+    <right_joint>front_right_wheel_joint</right_joint>
+    <wheel_separation>0.30</wheel_separation>
+    <wheel_radius>0.05</wheel_radius>
+    <topic>/cmd_vel</topic>
+    <odom_topic>/odom</odom_topic>
+    <tf_topic>/tf</tf_topic>
+    <odom_frame>odom</odom_frame>
+    <robot_base_frame>base_link</robot_base_frame>
+    <max_linear_acceleration>2.0</max_linear_acceleration>
+    <max_angular_acceleration>3.0</max_angular_acceleration>
+    <publish_odom>true</publish_odom>
+    <publish_tf>true</publish_tf>
+  </plugin>
+</gazebo>
+<gazebo>
+  <plugin
+      filename="gz-sim-diff-drive-system"
+      name="gz::sim::systems::DiffDrive">
+    <left_joint>rear_left_wheel_joint</left_joint>
+    <right_joint>rear_right_wheel_joint</right_joint>
+    <wheel_separation>0.30</wheel_separation>
+    <wheel_radius>0.05</wheel_radius>
+    <topic>/cmd_vel</topic>
+    <odom_topic>/odom</odom_topic>
+    <tf_topic>/tf</tf_topic>
+    <odom_frame>odom</odom_frame>
+    <robot_base_frame>base_link</robot_base_frame>
+    <max_linear_acceleration>2.0</max_linear_acceleration>
+    <max_angular_acceleration>3.0</max_angular_acceleration>
+    <publish_odom>true</publish_odom>
+    <publish_tf>true</publish_tf>
+  </plugin>
+</gazebo>
 </robot>

File: ros_ws/src/sumo/urdf/sumo.xacro (robot description, xacro)
@@ -1,9 +1,18 @@
 <?xml version="1.0"?>
 <robot xmlns:xacro="http://www.ros.org/wiki/xacro" name="sumo">
+  <link name="base_footprint">
+  <origin xyz="0.0 0.0 0.0"/>
+  </link>
+  <!-- <link name="box">
+    <visual>
+      <geometry>
+        <box size="0.357 0.369 0.145"/>
+      </geometry>
+    </visual>
+  </link> -->
   <link name="base_link">
     <visual>
-      <origin xyz="-0.17462 -0.18668 0" rpy="0 0 0"/>
-      <geometry>
-        <mesh filename="package://sumo/meshes/main-frame.STL" scale="0.001 0.001 0.001"/>
+      <geometry>
+        <mesh filename="package://sumo/meshes/blender frame trail 1.stl" scale="0.001 0.001 0.001"/>
       </geometry>
       <material name="gray">
@@ -12,29 +21,40 @@
     </visual>
     <collision>
-      <origin xyz="-0.17462 -0.18668 0" rpy="0 0 0"/>
-      <geometry>
-        <mesh filename="package://sumo/meshes/main-frame.STL" scale="0.001 0.001 0.001"/>
+      <!-- <origin xyz="-0.17462 -0.18668 0" rpy="0 0 0"/> -->
+      <geometry>
+        <!-- <mesh filename="package://sumo/meshes/blender frame trail 1.stl" scale="0.001 0.001 0.001"/> -->
+        <box size="0.345 0.37 0.145"/>
       </geometry>
     </collision>
    <inertial>
-    <origin xyz="-0.00117 0.00013 0.05125"/>
+    <!-- <origin xyz="-0.00117 0.00013 0.05125"/> -->
     <mass value="8.20158"/>
     <inertia ixx="0.0902089" ixy="0.0000740" ixz="0.0071159" iyy="0.0993226" iyz="0.0000221" izz="0.1666919"/>
   </inertial>
   </link>
+  <!-- <joint name="box_base_link_joint" type="fixed">
+    <parent link="base_link"/>
+    <child link="box"/>
+  </joint>  -->
+  <joint name="base_footprint_link_joint" type="fixed">
+    <parent link="base_footprint"/>
+    <child link="base_link"/>
+    <origin xyz="0.0 0.0 0.07"/>
+  </joint>
   <link name="rear_left_wheel_link">
     <visual>
-      <origin xyz="-0.03439 -0.03879 -0.05462" rpy="0 0 0"/>
-      <geometry>
-        <mesh filename="package://sumo/meshes/motor-wheel.STL" scale="0.001 0.001 0.001"/>
-      </geometry>
-      <material name="black">
-        <color rgba="0.1 0.1 0.1 1"/>
-      </material>
-    </visual>
-    <collision>
-      <origin xyz="-0.03439 -0.03879 -0.05462" rpy="0 0 0"/>
-      <geometry>
-        <mesh filename="package://sumo/meshes/motor-wheel.STL" scale="0.001 0.001 0.001"/>
+      <!-- <origin xyz="-0.03439 -0.03879 -0.05462" rpy="0 0 0"/> -->
+      <origin rpy="0.0 3.14159 0.0"/>
+      <geometry>
+        <mesh filename="package://sumo/meshes/motor B_L.stl" scale="0.001 0.001 0.001"/>
+      </geometry>
+      <material name="black">
+        <color rgba="0.1 0.1 0.1 1"/>
+      </material>
+    </visual>
+    <collision>
+      <origin xyz="0 0 0" rpy="1.57075 0 0"/>
+      <geometry>
+          <cylinder radius="0.065" length="0.027"/>
       </geometry>
     </collision>
@@ -48,21 +68,22 @@
     <parent link="base_link"/>
     <child link="rear_left_wheel_link"/>
-    <origin xyz="0.125 0.13775 0" rpy="0 0 0"/>
+    <origin xyz="-0.1166 0.142 -0.04" rpy="0 0 0"/>
     <axis xyz="0 1 0"/>
   </joint>
   <link name="rear_right_wheel_link">
     <visual>
-      <origin xyz="-0.03439 -0.03879 -0.05462" rpy="0 0 3.14159"/>
-      <geometry>
-        <mesh filename="package://sumo/meshes/motor-wheel.STL" scale="0.001 0.001 0.001"/>
-      </geometry>
-      <material name="black">
-        <color rgba="0.1 0.1 0.1 1"/>
-      </material>
-    </visual>
-    <collision>
-      <origin xyz="-0.03439 -0.03879 -0.05462" rpy="0 0 3.14159"/>
-      <geometry>
-        <mesh filename="package://sumo/meshes/motor-wheel.STL" scale="0.001 0.001 0.001"/>
+    <origin rpy="3.1415 -3.1415 0.0"/>
+      <!-- <origin xyz="-0.03439 -0.03879 -0.05462" rpy="0 0 3.14159"/> -->
+      <geometry>
+        <mesh filename="package://sumo/meshes/motor B_R.stl" scale="0.001 0.001 0.001"/>
+      </geometry>
+      <material name="black">
+        <color rgba="0.1 0.1 0.1 1"/>
+      </material>
+    </visual>
+    <collision>
+      <origin xyz="0 0 0" rpy="1.57075 0 0"/>
+      <geometry>
+          <cylinder radius="0.065" length="0.027"/>
       </geometry>
     </collision>
@@ -76,21 +97,22 @@
     <parent link="base_link"/>
     <child link="rear_right_wheel_link"/>
-    <origin xyz="0.125 -0.13775 0" rpy="0 0 0"/>
+    <origin xyz="-0.117 -0.1425 -0.04" rpy="0 0 0"/>
     <axis xyz="0 1 0"/>
   </joint>
   <link name="front_left_wheel_link">
     <visual>
-      <origin xyz="-0.03439 -0.03879 -0.05462" rpy="0 0 0"/>
-      <geometry>
-        <mesh filename="package://sumo/meshes/motor-wheel.STL" scale="0.001 0.001 0.001"/>
-      </geometry>
-      <material name="black">
-        <color rgba="0.1 0.1 0.1 1"/>
-      </material>
-    </visual>
-    <collision>
-      <origin xyz="-0.03439 -0.03879 -0.05462" rpy="0 0 0"/>
-      <geometry>
-        <mesh filename="package://sumo/meshes/motor-wheel.STL" scale="0.001 0.001 0.001"/>
+      <!-- <origin xyz="-0.03439 -0.03879 -0.05462" rpy="0 0 0"/> -->
+      <!-- <origin rpy="3.1415 0.0 0.0"/> -->
+      <geometry>
+        <mesh filename="package://sumo/meshes/MOTOR-FL.stl" scale="0.001 0.001 0.001"/>
+      </geometry>
+      <material name="black">
+        <color rgba="0.1 0.1 0.1 1"/>
+      </material>
+    </visual>
+    <collision>
+      <origin xyz="0 0 0" rpy="1.57075 0 0"/>
+      <geometry>
+          <cylinder radius="0.065" length="0.027"/>
       </geometry>
     </collision>
@@ -104,21 +126,22 @@
     <parent link="base_link"/>
     <child link="front_left_wheel_link"/>
-    <origin xyz="-0.125 0.13775 0" rpy="0 0 0"/>
+    <origin xyz="0.034 0.142 -0.04" rpy="0 0 0"/>
     <axis xyz="0 1 0"/>
   </joint>
   <link name="front_right_wheel_link">
     <visual>
-      <origin xyz="-0.03439 -0.03879 -0.05462" rpy="0 0 3.14159"/>
-      <geometry>
-        <mesh filename="package://sumo/meshes/motor-wheel.STL" scale="0.001 0.001 0.001"/>
-      </geometry>
-      <material name="black">
-        <color rgba="0.1 0.1 0.1 1"/>
-      </material>
-    </visual>
-    <collision>
-      <origin xyz="-0.03439 -0.03879 -0.05462" rpy="0 0 3.14159"/>
-      <geometry>
-        <mesh filename="package://sumo/meshes/motor-wheel.STL" scale="0.001 0.001 0.001"/>
+    <!-- <origin rpy="3.1415 0.0 0.0"/> -->
+      <!-- <origin xyz="-0.03439 -0.03879 -0.05462" rpy="0 0 3.14159"/> -->
+      <geometry>
+        <mesh filename="package://sumo/meshes/motor F_R.stl" scale="0.001 0.001 0.001"/>
+      </geometry>
+      <material name="black">
+        <color rgba="0.1 0.1 0.1 1"/>
+      </material>
+    </visual>
+    <collision>
+      <origin xyz="0 0 0" rpy="1.57075 0 0"/>
+      <geometry>
+          <cylinder radius="0.065" length="0.027"/>
       </geometry>
     </collision>
@@ -132,12 +155,12 @@
     <parent link="base_link"/>
     <child link="front_right_wheel_link"/>
-    <origin xyz="-0.125 -0.13775 0" rpy="0 0 0"/>
-    <axis xyz="0 1 0"/>
-  </joint>
-  <link name="lidar_link">
-    <visual>
-      <origin xyz="-0.07142 -0.06488 -0.09997" rpy="1.57075 0.0 0.0"/>
-      <geometry>
-        <mesh filename="package://sumo/meshes/lidar.STL" scale="0.001 0.001 0.001"/>
+    <origin xyz="0.0335 -0.1425 -0.04" rpy="0 0 0"/>
+    <axis xyz="0 1 0"/>
+  </joint>
+  <link name="lidar_mesh_link">
+    <visual>
+      <!-- <origin xyz="0.10 0.10 -0.09997" rpy="1.57075 0 0"/> -->
+      <geometry>
+        <mesh filename="package://sumo/meshes/lidar blender trial1.stl" scale="0.001 0.001 0.001"/>
       </geometry>
       <material name="blue">
@@ -146,7 +169,7 @@
     </visual>
     <collision>
-      <origin xyz="-0.07142 -0.06488 -0.09997" rpy="1.57075 0.0 0.0"/>
-      <geometry>
-        <mesh filename="package://sumo/meshes/lidar.STL" scale="0.001 0.001 0.001"/>
+      <!-- <origin xyz="0.10 0.10 -0.09997" rpy="1.57075 0 0"/> -->
+      <geometry>
+        <box size="0.075 0.07 0.063"/>
       </geometry>
     </collision>
@@ -157,14 +180,21 @@
     </inertial>
   </link>
-  <joint name="lidar_joint" type="fixed">
-    <parent link="base_link"/>
-    <child link="lidar_link"/>
-    <origin xyz="-0.08177 0 0.170" rpy="0 0 0"/>
+  <link name="lidar_link">
+  </link>
+  <joint name="lidar_link_joint" type="fixed">
+  <parent link="lidar_mesh_link"/>
+  <child link="lidar_link"/>
+    <origin xyz="0.0 0.0 0.037"/>
+  </joint>
+  <joint name="lidar_mesh_joint" type="fixed">
+    <parent link="base_link"/>
+    <child link="lidar_mesh_link"/>
+    <origin xyz="-0.096 0 0.0737" rpy="0 0 0"/>
   </joint>
   <link name="camera_link">
     <visual>
-      <origin xyz="-0.03889 0.1 -0.04598" rpy="1.57075 0 -1.57075"/>
-      <geometry>
-        <mesh filename="package://sumo/meshes/camera.STL" scale="0.001 0.001 0.001"/>
+      <!-- <origin xyz="-0.03889 0.03714 -0.03598" rpy="1.5708 0 -1.5708"/> -->
+      <geometry>
+        <mesh filename="package://sumo/meshes/blender trial cam .stl" scale="0.001 0.001 0.001"/>
       </geometry>
       <material name="white">
@@ -173,7 +203,8 @@
     </visual>
     <collision>
-      <origin xyz="-0.03889 -0.02314 -0.02598" rpy="0 0 0"/>
-      <geometry>
-        <mesh filename="package://sumo/meshes/camera.STL" scale="0.001 0.001 0.001"/>
+      <!-- <origin xyz="-0.03889 0.03714 -0.03598" rpy="1.5708 0 -1.5708"/> -->
+      <geometry>
+        <!-- <mesh filename="package://sumo/meshes/blender trial cam .stl" scale="0.001 0.001 0.001"/> -->
+        <box size="0.02 0.077 0.025"/>
       </geometry>
     </collision>
@@ -187,5 +218,6 @@
     <parent link="base_link"/>
     <child link="camera_link"/>
-    <origin xyz="0.02870 0 0.13220" rpy="0 0 0"/>
-  </joint>
+    <origin xyz="0.031 0 0.047" rpy="0 0 0"/>
+  </joint>
+<xacro:include filename="gazebo.xacro"/>
 </robot>
